Commit message: Update adam_assem1.urdf

File: urdf/adam_assem1.urdf (robot description, URDF)
Before this commit: robot Adam_Assem1, 5 links, 4 joints
Links:
- link base_link: geometry collision mesh filename=package://adam_assem1/meshes/base_link.STL; visual mesh filename=package://adam_assem1/meshes/base_link.STL
- link front_wheel1: geometry collision mesh filename=package://adam_assem1/meshes/front_wheel1.STL; visual mesh filename=package://adam_assem1/meshes/front_wheel1.STL
- link front_wheel2: geometry collision mesh filename=package://adam_assem1/meshes/front_wheel2.STL; visual mesh filename=package://adam_assem1/meshes/front_wheel2.STL
- link rear_wheel1: geometry collision mesh filename=package://adam_assem1/meshes/rear_wheel1.STL; visual mesh filename=package://adam_assem1/meshes/rear_wheel1.STL
- link rear_wheel2: geometry collision mesh filename=package://adam_assem1/meshes/rear_wheel2.STL; visual mesh filename=package://adam_assem1/meshes/rear_wheel2.STL
